File: tht-dip.sch (KiCad schematic (older format))
At the start: 55 parts, among them J1 Conn_01x01_Female, J10 Conn_01x01_Female, J2 Conn_01x01_Female, J3 Conn_01x01_Female, J4 Conn_01x01_Female, J5 Conn_01x01_Female, J6 Conn_01x01_Female, J7 Conn_01x01_Female, J8 Conn_01x01_Female, J9 Conn_01x01_Female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

Commit message: Add files via upload
Parts:
- removed R19, R27: 8K, Resistor_THT:R_Axial_DIN0204_L3.6mm_D1.6mm_P5.08mm_Horizontal, symbol Device:R
- R13, R21: value 2K -> 3K
- R14, R22: value 3K -> 4K
- R15, R23: value 4K -> 5K
- R16, R24: value 5K -> 6K
- R17, R25: value 6K -> 7K
- R18, R26: value 7K -> 8K
Connections:
- no-connect marks 6 -> 8
Changed lines of the file:
@@
 P 3600 5000
 F 0 "R13" V 3600 5000 50  0000 C CNN
-F 1 "2K" V 3550 5200 50  0000 C CNN
+F 1 "3K" V 3550 5200 50  0000 C CNN
 F 2 "Resistor_THT:R_Axial_DIN0204_L3.6mm_D1.6mm_P5.08mm_Horizontal" V 3530 5000 50  0001 C CNN
 F 3 "~" H 3600 5000 50  0001 C CNN
@@
 P 3600 5100
 F 0 "R14" V 3600 5100 50  0000 C CNN
-F 1 "3K" V 3550 5300 50  0000 C CNN
+F 1 "4K" V 3550 5300 50  0000 C CNN
 F 2 "Resistor_THT:R_Axial_DIN0204_L3.6mm_D1.6mm_P5.08mm_Horizontal" V 3530 5100 50  0001 C CNN
 F 3 "~" H 3600 5100 50  0001 C CNN
@@
 P 3600 5200
 F 0 "R15" V 3600 5200 50  0000 C CNN
-F 1 "4K" V 3550 5400 50  0000 C CNN
+F 1 "5K" V 3550 5400 50  0000 C CNN
 F 2 "Resistor_THT:R_Axial_DIN0204_L3.6mm_D1.6mm_P5.08mm_Horizontal" V 3530 5200 50  0001 C CNN
 F 3 "~" H 3600 5200 50  0001 C CNN
@@
 P 3600 5300
 F 0 "R16" V 3600 5300 50  0000 C CNN
-F 1 "5K" V 3550 5500 50  0000 C CNN
+F 1 "6K" V 3550 5500 50  0000 C CNN
 F 2 "Resistor_THT:R_Axial_DIN0204_L3.6mm_D1.6mm_P5.08mm_Horizontal" V 3530 5300 50  0001 C CNN
 F 3 "~" H 3600 5300 50  0001 C CNN
@@
 P 3600 5400
 F 0 "R17" V 3600 5400 50  0000 C CNN
-F 1 "6K" V 3550 5600 50  0000 C CNN
+F 1 "7K" V 3550 5600 50  0000 C CNN
 F 2 "Resistor_THT:R_Axial_DIN0204_L3.6mm_D1.6mm_P5.08mm_Horizontal" V 3530 5400 50  0001 C CNN
 F 3 "~" H 3600 5400 50  0001 C CNN
@@
 P 3600 5500
 F 0 "R18" V 3600 5500 50  0000 C CNN
-F 1 "7K" V 3550 5700 50  0000 C CNN
+F 1 "8K" V 3550 5700 50  0000 C CNN
 F 2 "Resistor_THT:R_Axial_DIN0204_L3.6mm_D1.6mm_P5.08mm_Horizontal" V 3530 5500 50  0001 C CNN
 F 3 "~" H 3600 5500 50  0001 C CNN
@@
 	0    1    1    0
 $EndComp
-$Comp
-L Device:R R19
-U 1 1 60E3C240
-P 3600 5600
-F 0 "R19" V 3600 5600 50  0000 C CNN
-F 1 "8K" V 3550 5800 50  0000 C CNN
-F 2 "Resistor_THT:R_Axial_DIN0204_L3.6mm_D1.6mm_P5.08mm_Horizontal" V 3530 5600 50  0001 C CNN
-F 3 "~" H 3600 5600 50  0001 C CNN
-	1    3600 5600
-	0    1    1    0
-$EndComp
-Wire Wire Line
-	3750 5600 3750 5500
 Wire Wire Line
 	3750 5500 3750 5400
-Connection ~ 3750 5500
 Wire Wire Line
 	3750 5400 3750 5300
@@
 Wire Wire Line
 	3250 5500 3450 5500
-Wire Wire Line
-	3250 5600 3450 5600
 Wire Wire Line
 	2650 5600 2650 5500
@@
 P 3600 6500
 F 0 "R21" V 3600 6500 50  0000 C CNN
-F 1 "2K" V 3550 6700 50  0000 C CNN
+F 1 "3K" V 3550 6700 50  0000 C CNN
 F 2 "Resistor_THT:R_Axial_DIN0204_L3.6mm_D1.6mm_P5.08mm_Horizontal" V 3530 6500 50  0001 C CNN
 F 3 "~" H 3600 6500 50  0001 C CNN
@@
 P 3600 6600
 F 0 "R22" V 3600 6600 50  0000 C CNN
-F 1 "3K" V 3550 6800 50  0000 C CNN
+F 1 "4K" V 3550 6800 50  0000 C CNN
 F 2 "Resistor_THT:R_Axial_DIN0204_L3.6mm_D1.6mm_P5.08mm_Horizontal" V 3530 6600 50  0001 C CNN
 F 3 "~" H 3600 6600 50  0001 C CNN
@@
 P 3600 6700
 F 0 "R23" V 3600 6700 50  0000 C CNN
-F 1 "4K" V 3550 6900 50  0000 C CNN
+F 1 "5K" V 3550 6900 50  0000 C CNN
 F 2 "Resistor_THT:R_Axial_DIN0204_L3.6mm_D1.6mm_P5.08mm_Horizontal" V 3530 6700 50  0001 C CNN
 F 3 "~" H 3600 6700 50  0001 C CNN
@@
 P 3600 6800
 F 0 "R24" V 3600 6800 50  0000 C CNN
-F 1 "5K" V 3550 7000 50  0000 C CNN
+F 1 "6K" V 3550 7000 50  0000 C CNN
 F 2 "Resistor_THT:R_Axial_DIN0204_L3.6mm_D1.6mm_P5.08mm_Horizontal" V 3530 6800 50  0001 C CNN
 F 3 "~" H 3600 6800 50  0001 C CNN
@@
 P 3600 6900
 F 0 "R25" V 3600 6900 50  0000 C CNN
-F 1 "6K" V 3550 7100 50  0000 C CNN
+F 1 "7K" V 3550 7100 50  0000 C CNN
 F 2 "Resistor_THT:R_Axial_DIN0204_L3.6mm_D1.6mm_P5.08mm_Horizontal" V 3530 6900 50  0001 C CNN
 F 3 "~" H 3600 6900 50  0001 C CNN
@@
 P 3600 7000
 F 0 "R26" V 3600 7000 50  0000 C CNN
-F 1 "7K" V 3550 7200 50  0000 C CNN
+F 1 "8K" V 3550 7200 50  0000 C CNN
 F 2 "Resistor_THT:R_Axial_DIN0204_L3.6mm_D1.6mm_P5.08mm_Horizontal" V 3530 7000 50  0001 C CNN
 F 3 "~" H 3600 7000 50  0001 C CNN
@@
 	0    1    1    0
 $EndComp
-$Comp
-L Device:R R27
-U 1 1 60EB3DF3
-P 3600 7100
-F 0 "R27" V 3600 7100 50  0000 C CNN
-F 1 "8K" V 3550 7300 50  0000 C CNN
-F 2 "Resistor_THT:R_Axial_DIN0204_L3.6mm_D1.6mm_P5.08mm_Horizontal" V 3530 7100 50  0001 C CNN
-F 3 "~" H 3600 7100 50  0001 C CNN
-	1    3600 7100
-	0    1    1    0
-$EndComp
-Wire Wire Line
-	3750 7100 3750 7000
 Wire Wire Line
 	3750 7000 3750 6900
-Connection ~ 3750 7000
 Wire Wire Line
 	3750 6900 3750 6800
@@
 Wire Wire Line
 	3250 7000 3450 7000
-Wire Wire Line
-	3250 7100 3450 7100
 Wire Wire Line
 	2650 7100 2650 7000
@@
 	4450 1250 4900 1250
 Connection ~ 4900 1250
+NoConn ~ 3250 5600
+NoConn ~ 3250 7100
 $EndSCHEMATC

Commit message: Add files via upload
Parts:
- removed C3: 33uF, Capacitor_THT:C_Disc_D5.0mm_W2.5mm_P2.50mm, symbol Device:C
- added C3: 33uF, Capacitor_THT:CP_Radial_D6.3mm_P2.50mm, symbol Device:CP
Connections:
- net GND: now also C3.2
- net VCC: now also C3.1
Changed lines of the file:
@@
 Connection ~ 7350 1850
-$Comp
-L Device:C C3
-U 1 1 60CCFCFB
-P 5800 1100
-F 0 "C3" H 5915 1146 50  0000 L CNN
-F 1 "33uF" H 5915 1055 50  0000 L CNN
-F 2 "Capacitor_THT:C_Disc_D5.0mm_W2.5mm_P2.50mm" H 5838 950 50  0001 C CNN
-F 3 "~" H 5800 1100 50  0001 C CNN
-	1    5800 1100
-	1    0    0    -1
-$EndComp
 $Comp
 L Device:R R1
@@
 	6550 950  6550 1550
 Wire Wire Line
-	6150 950  5800 950
-Wire Wire Line
-	5800 950  5400 950
-Connection ~ 5800 950
-Wire Wire Line
 	5400 950  4900 950
 Connection ~ 5400 950
@@
 	5400 1250 5800 1250
 Connection ~ 5400 1250
-Connection ~ 5800 1250
 Text GLabel 4900 900  1    50   Input ~ 0
 VCC
@@
 NoConn ~ 3250 5600
 NoConn ~ 3250 7100
+Wire Wire Line
+	5400 950  5800 950
+$Comp
+L Device:CP C3
+U 1 1 60E42580
+P 5800 1100
+F 0 "C3" H 5918 1146 50  0000 L CNN
+F 1 "33uF" H 5918 1055 50  0000 L CNN
+F 2 "Capacitor_THT:CP_Radial_D6.3mm_P2.50mm" H 5838 950 50  0001 C CNN
+F 3 "~" H 5800 1100 50  0001 C CNN
+	1    5800 1100
+	1    0    0    -1
+$EndComp
+Connection ~ 5800 950
+Wire Wire Line
+	5800 950  6150 950
+Connection ~ 5800 1250
 $EndSCHEMATC
