File: tht-dip.sch (KiCad schematic (older format))
At the start: 55 parts, among them J1 Conn_01x01_Female, J10 Conn_01x01_Female, J2 Conn_01x01_Female, J3 Conn_01x01_Female, J4 Conn_01x01_Female, J5 Conn_01x01_Female, J6 Conn_01x01_Female, J7 Conn_01x01_Female, J8 Conn_01x01_Female, J9 Conn_01x01_Female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

Commit message: Add files via upload
Changed to TL082BCP , less current use.
Parts:
- removed U1, U2: NE5534, Package_DIP:DIP-8_W7.62mm_Socket, symbol Amplifier_Operational:NE5534
- added U1: TL082BCP, Package_DIP:DIP-8_W7.62mm, symbol Amplifier_Operational:TL082
- D1: value 1N4746A (18V) -> 1N5241B-TR
Connections:
- net GND: now also U1.4 (V-)
- net ResIN: now also U1.2 (-)
- net ResIN1: now also U1.6 (-)
- net ResOUT: now also U1.1
- net ResOUT2: now also U1.7
- net VCC: now also U1.8 (V+)
- net ind: now also U1.5 (+)
- net at D4.2 (A), D5.1 (K), J4.1 (Pin_1)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: now also U1.3 (+)
- no-connect marks 6 -> 0
Other:
- note added: "ZENER 11V 500MW DO35"
Changed lines of the file:
@@
 P 6550 1700
 F 0 "D1" V 6504 1780 50  0000 L CNN
-F 1 "1N4746A (18V)" V 6595 1780 50  0000 L CNN
+F 1 "1N5241B-TR" V 6595 1780 50  0000 L CNN
 F 2 "Diode_THT:D_DO-35_SOD27_P7.62mm_Horizontal" H 6550 1700 50  0001 C CNN
 F 3 "~" H 6550 1700 50  0001 C CNN
@@
 Text GLabel 4900 900  1    50   Input ~ 0
 VCC
-Text GLabel 4950 2050 1    50   Input ~ 0
+Text GLabel 6800 3350 1    50   Input ~ 0
 VCC
 Wire Wire Line
-	4950 2050 4950 2200
+	6800 3350 6800 3500
 Connection ~ 4900 950
 Wire Wire Line
@@
 	0    1    1    0
 $EndComp
-NoConn ~ 5050 2200
-NoConn ~ 5050 2800
-NoConn ~ 5150 2800
-Text GLabel 4950 2900 3    50   Input ~ 0
+Text GLabel 6800 4200 3    50   Input ~ 0
 V-
 Wire Wire Line
-	4950 2900 4950 2800
+	6800 4200 6800 4100
 $Comp
 L Device:R R4
@@
 	3600 3250 3600 3500
 Connection ~ 7350 2700
-$Comp
-L Amplifier_Operational:NE5534 U1
-U 1 1 60CCF692
-P 5050 2500
-F 0 "U1" H 5394 2546 50  0000 L CNN
-F 1 "NE5534" H 5394 2455 50  0000 L CNN
-F 2 "Package_DIP:DIP-8_W7.62mm_Socket" H 5100 2550 50  0001 C CNN
-F 3 "http://www.ti.com/lit/ds/symlink/ne5534.pdf" H 5100 2650 50  0001 C CNN
-	1    5050 2500
-	1    0    0    -1
-$EndComp
 Wire Wire Line
 	7200 2700 7350 2700
@@
 Wire Wire Line
 	5350 2500 5750 2500
-Connection ~ 5350 2500
 $Comp
 L Device:R R9
@@
 Connection ~ 3600 1250
 Connection ~ 8400 3050
-Text GLabel 5700 3500 1    50   Input ~ 0
-VCC
-Wire Wire Line
-	5700 3500 5700 3650
-NoConn ~ 5800 4250
-Text GLabel 5700 4350 3    50   Input ~ 0
-V-
-Wire Wire Line
-	5700 4350 5700 4250
 Wire Wire Line
 	5500 4050 5500 4700
@@
 	6050 4200 6100 4200
 Wire Wire Line
-	6100 4200 6100 3950
-Wire Wire Line
 	6550 2700 6100 2700
-Wire Wire Line
-	6100 2700 6100 3950
-Connection ~ 6100 3950
 Connection ~ 3600 3500
 Wire Wire Line
@@
 Wire Wire Line
 	4650 2600 4750 2600
-$Comp
-L Amplifier_Operational:NE5534 U2
-U 1 1 60D5461E
-P 5800 3950
-F 0 "U2" H 6144 3996 50  0000 L CNN
-F 1 "NE5534" H 6144 3905 50  0000 L CNN
-F 2 "Package_DIP:DIP-8_W7.62mm_Socket" H 5850 4000 50  0001 C CNN
-F 3 "http://www.ti.com/lit/ds/symlink/ne5534.pdf" H 5850 4100 50  0001 C CNN
-	1    5800 3950
-	1    0    0    -1
-$EndComp
 Text Notes 8650 2700 0    50   ~ 0
 +48 V phantom power
@@
 Wire Wire Line
 	1900 1550 2800 1550
-NoConn ~ 5800 3650
-NoConn ~ 5900 4250
 $Comp
 L Device:D D2
@@
 Wire Wire Line
 	5050 4050 5500 4050
-Connection ~ 5500 4050
 $Comp
 L power:GND #PWR07
@@
 Wire Wire Line
 	3450 4900 3250 4900
+Wire Wire Line
+	6100 2700 6100 3950
+$Comp
+L Amplifier_Operational:TL082 U1
+U 1 1 60F62BF2
+P 5050 2500
+F 0 "U1" H 5050 2867 50  0000 C CNN
+F 1 "TL082BCP " H 5050 2776 50  0000 C CNN
+F 2 "Package_DIP:DIP-8_W7.62mm" H 5050 2500 50  0001 C CNN
+F 3 "http://www.ti.com/lit/ds/symlink/tl081.pdf" H 5050 2500 50  0001 C CNN
+	1    5050 2500
+	1    0    0    -1
+$EndComp
+Connection ~ 5350 2500
+$Comp
+L Amplifier_Operational:TL082 U1
+U 2 1 60F66AC4
+P 5800 3950
+F 0 "U1" H 5800 4317 50  0000 C CNN
+F 1 "TL082BCP " H 5800 4226 50  0000 C CNN
+F 2 "Package_DIP:DIP-8_W7.62mm" H 5800 3950 50  0001 C CNN
+F 3 "http://www.ti.com/lit/ds/symlink/tl081.pdf" H 5800 3950 50  0001 C CNN
+	2    5800 3950
+	1    0    0    -1
+$EndComp
+Connection ~ 6100 3950
+Wire Wire Line
+	6100 3950 6100 4200
+Connection ~ 5500 4050
+$Comp
+L Amplifier_Operational:TL082 U1
+U 3 1 60F6BF6F
+P 6900 3800
+F 0 "U1" H 6858 3846 50  0000 L CNN
+F 1 "TL082BCP " H 6858 3755 50  0000 L CNN
+F 2 "Package_DIP:DIP-8_W7.62mm" H 6900 3800 50  0001 C CNN
+F 3 "http://www.ti.com/lit/ds/symlink/tl081.pdf" H 6900 3800 50  0001 C CNN
+	3    6900 3800
+	1    0    0    -1
+$EndComp
+Text Notes 5500 1750 0    50   ~ 0
+ZENER 11V 500MW DO35
 $EndSCHEMATC
