File: tht-dip.kicad_sch (KiCad schematic)
At the start: 54 parts, among them J1 Conn_01x01_Female, J10 Conn_01x01_Female, J2 Conn_01x01_Female, J3 Conn_01x01_Female, J4 Conn_01x01_Female, J5 Conn_01x01_Female, J6 Conn_01x01_Female, J7 Conn_01x01_Female, J8 Conn_01x01_Female, J9 Conn_01x01_Female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

Commit message: Add files via upload
Parts:
- removed R12, R20: 1K, Resistor_THT:R_Axial_DIN0204_L3.6mm_D1.6mm_P5.08mm_Horizontal, symbol Device:R
- removed R13, R21: 3K, Resistor_THT:R_Axial_DIN0204_L3.6mm_D1.6mm_P5.08mm_Horizontal, symbol Device:R
- removed R14, R22: 4K, Resistor_THT:R_Axial_DIN0204_L3.6mm_D1.6mm_P5.08mm_Horizontal, symbol Device:R
- removed R15, R23: 5K, Resistor_THT:R_Axial_DIN0204_L3.6mm_D1.6mm_P5.08mm_Horizontal, symbol Device:R
- removed R16, R24: 6K, Resistor_THT:R_Axial_DIN0204_L3.6mm_D1.6mm_P5.08mm_Horizontal, symbol Device:R
- removed R17, R25: 7K, Resistor_THT:R_Axial_DIN0204_L3.6mm_D1.6mm_P5.08mm_Horizontal, symbol Device:R
- removed R18, R26: 8K, Resistor_THT:R_Axial_DIN0204_L3.6mm_D1.6mm_P5.08mm_Horizontal, symbol Device:R
- removed R19, R27: 700, Resistor_THT:R_Axial_DIN0204_L3.6mm_D1.6mm_P5.08mm_Horizontal, symbol Device:R
- removed SW1, SW2: JS0108AP4-S, Package_DIP:DIP-16_W7.62mm, symbol Switch:SW_DIP_x08
- added RV1: PTD902-2015K-B103, potmeter:PTD902-2015K-B103, symbol Device:R_Potentiometer_Dual
- C1: renamed from C9; footprint Capacitor_THT:C_Disc_D5.0mm_W2.5mm_P2.50mm -> Capacitor_THT:CP_Radial_D5.0mm_P2.00mm
- C7: renamed from C6; footprint Capacitor_THT:C_Disc_D5.0mm_W2.5mm_P2.50mm -> Capacitor_THT:CP_Radial_D5.0mm_P2.00mm
- C9: renamed from C8; footprint Capacitor_THT:C_Disc_D5.0mm_W2.5mm_P2.50mm -> Capacitor_THT:CP_Radial_D5.0mm_P2.00mm
- renumbered C1 to C2, C2 to C3, C3 to C4, C4 to C5, C5 to C6, C7 to C8
Connections:
- net ResIN: now also RV1.1
- net ResIN1: now also RV1.4
- net ResOUT: now also RV1.2
- net ResOUT2: now also RV1.5
- no-connect marks 0 -> 2
Other:
- note removed: "SW1 and SW2 switch setting, Gain values in dB: 700=18 1K=20 3K=29 4K=32 5K=34 6K=35 7K=37 8K=38 Both must be set to the same."
